File: base.brd (EAGLE design)
At the start: 64.8 x 71.1 mm, 67 parts

Commit message: Version 2 shark prototype boards
Parts:
- removed D4, D5: (no value), tekdemo:WS2812B
- removed I2C: (no value), SparkFun-Connectors:1X04
- removed I2C_SERVO_DIVER: (no value), adafruit:TSSOP28
- removed J_BITE, J_DRVL, J_DRVR, J_FINL, J_FINR, J_TAIL: (no value), SparkFun-Passives:PAD-JUMPER-2-NO_YES_SILK
- removed J_EXT_CLK: CLK2GND, SparkFun-Retired:SJ_2S-TRACE
- removed RI2CA, RI2CL: 430, tekdemo:0402-0603-0805-UNIVERSAL
- added BP_P1, BP_P2, BP_P3: (no value), SparkFun-Passives:PAD-JUMPER-2-NO_YES_SILK
- moved LOGO1 19.3 mm to (55.9, 26.7)
- moved C_S1 18.6 mm to (70.1, 50.0), turned to 0 degrees
- moved C_S2 16.2 mm to (70.1, 48.0), turned to 0 degrees
- moved WS_OUT 14.0 mm to (90.2, 24.9)
- moved DRV_L 14.0 mm to (66.8, 26.7)
- moved DRV_R 14.0 mm to (66.8, 29.2)
- moved FIN_L 14.0 mm to (66.8, 31.8)
- moved FIN_R 14.0 mm to (66.8, 36.8)
- moved TAIL 14.0 mm to (66.8, 39.4)
- moved BITE 14.0 mm to (66.8, 41.9)
- moved C_S3 13.7 mm to (70.1, 45.7), turned to 0 degrees
- moved C_BLKY 1.52 mm to (92.7, 51.8)
Connections:
- removed net BITE: BITE.1, I2C_SERVO_DIVER.11, J_BITE.2
- removed net DRVL: DRV_L.1, I2C_SERVO_DIVER.6, J_DRVL.2
- removed net DRVR: DRV_R.1, I2C_SERVO_DIVER.7, J_DRVR.2
- removed net FINL: FIN_L.1, I2C_SERVO_DIVER.8, J_FINL.2
- removed net FINR: FIN_R.1, I2C_SERVO_DIVER.9, J_FINR.2
- removed net I2C_SCL: I2C.4, I2C_SERVO_DIVER.26, J_BITE.1, RI2CA.-, X1.13
- removed net I2C_SDA: I2C.3, I2C_SERVO_DIVER.27, J_TAIL.1, RI2CL.-, X1.14
- removed net N$13: D4.2, D5.4
- removed net N$14: D5.2, WS_OUT.2
- removed net N$2: I2C_SERVO_DIVER.25, J_EXT_CLK.2
- removed net TAIL: I2C_SERVO_DIVER.10, J_TAIL.2, TAIL.1
- new net 4: TAIL.1, X1.14
- new net 5: BITE.1, X1.13
- net 12: now also FIN_L.1; no longer J_FINL.1
- net 13: now also FIN_R.1; no longer I2C_SERVO_DIVER.23, J_FINR.1
- net 14: now also DRV_R.1; no longer J_DRVR.1
- net 16: now also DRV_L.1; no longer J_DRVL.1
- net 3.0V: no longer I2C.2, I2C_SERVO_DIVER.28, RI2CA.+, RI2CL.+
- net ESP_RX_I: now also UART_X.TX_B; no longer UART_X.RX_B
- net ESP_TX_O: now also UART_X.RX_B; no longer UART_X.TX_B
- net GND: no longer D4.3, D5.3, I2C.1, I2C_SERVO_DIVER.1, I2C_SERVO_DIVER.14, I2C_SERVO_DIVER.2, I2C_SERVO_DIVER.24, I2C_SERVO_DIVER.3, I2C_SERVO_DIVER.4, I2C_SERVO_DIVER.5, J_EXT_CLK.1
- net N$10: now also BP_P1.1
- net N$11: now also BP_P2.2, BP_P3.1
- net N$12: now also BP_P3.2, WS_OUT.2; no longer D4.4
- net N$3: now also BP_P1.2, BP_P2.1
- net VSUPPLY: no longer D4.1, D5.1
Routing:
- net I2C_SCL: track 75.5 -> 0.00 mm, vias 2 -> 0
- net DRVL: track 70.1 -> 0.00 mm
- net I2C_SDA: track 68.6 -> 0.00 mm
- net DRVR: track 64.8 -> 0.00 mm
- net FINL: track 58.5 -> 0.00 mm
- net FINR: track 49.5 -> 0.00 mm
- net TAIL: track 44.2 -> 0.00 mm
- net N$16: track 42.1 -> 0.00 mm
- net 4: track 0.00 -> 41.2 mm
- net BITE: track 40.4 -> 0.00 mm
- net N$18: track 30.5 -> 0.00 mm
- net 3.0V: track 125.5 -> 95.6 mm, vias 8 -> 6
- net 5: track 0.00 -> 29.2 mm
- net 13: track 58.4 -> 34.1 mm, vias 4 -> 2
- net GND: track 104.8 -> 86.4 mm, vias 54 -> 46
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Other:
- board size 64.8 x 71.1 mm -> 64.8 x 57.2 mm
- board text added: "+ S -"
- board text removed: "HI KELLY! Hi GABE! :D"
- board text removed: "UART FOOTPRINT IS CURRENTLY LOOPBACK OR STRAIGHT. FIX"
- board text removed: "UART FOOTPRINT NEEDS TO BE FURTHER OUT AND/OR WIDER PADS"
- board text removed: "WAFFLES!"
