File: base.sch (EAGLE design)
At the start: 67 parts

Commit message: Version 2 shark prototype boards
Parts:
- removed D4, D5: (no value), tekdemo:WS2812B
- removed I2C: (no value), SparkFun-Connectors:I2C_STANDARD
- removed I2C_SERVO_DIVER: (no value), adafruit:PCA9685
- removed J_BITE, J_DRVL, J_DRVR, J_FINL, J_FINR, J_TAIL: JUMPER-PAD-2-NOYES_SILK, SparkFun-Passives:JUMPER-PAD-2-NOYES_SILK
- removed J_EXT_CLK: CLK2GND, SparkFun-Retired:SOLDERJUMPERTRACE
- removed RI2CA, RI2CL: 430, tekdemo:RESISTORUNIVERSAL
- added BP_P1, BP_P2, BP_P3: JUMPER-PAD-2-NOYES_SILK, SparkFun-Passives:JUMPER-PAD-2-NOYES_SILK
Connections:
- removed net BITE: BITE.1, I2C_SERVO_DIVER.PWM5, J_BITE.2
- removed net DRVL: DRV_L.1, I2C_SERVO_DIVER.PWM0, J_DRVL.2
- removed net DRVR: DRV_R.1, I2C_SERVO_DIVER.PWM1, J_DRVR.2
- removed net FINL: FIN_L.1, I2C_SERVO_DIVER.PWM2, J_FINL.2
- removed net FINR: FIN_R.1, I2C_SERVO_DIVER.PWM3, J_FINR.2
- removed net I2C_SCL: I2C.4, I2C_SERVO_DIVER.SCL, J_BITE.1, RI2CA.2, X1.GPIO5
- removed net I2C_SDA: I2C.3, I2C_SERVO_DIVER.SDA, J_TAIL.1, RI2CL.2, X1.GPIO4
- removed net N$13: D4.DOUT, D5.DIN
- removed net N$14: D5.DOUT, WS_OUT.2
- removed net N$2: I2C_SERVO_DIVER.EXTCLK, J_EXT_CLK.2
- removed net TAIL: I2C_SERVO_DIVER.PWM4, J_TAIL.2, TAIL.1
- new net 4: TAIL.1, X1.GPIO4
- new net 5: BITE.1, X1.GPIO5
- net 12: now also FIN_L.1; no longer J_FINL.1
- net 13: now also FIN_R.1; no longer I2C_SERVO_DIVER.#OE, J_FINR.1
- net 14: now also DRV_R.1; no longer J_DRVR.1
- net 16: now also DRV_L.1; no longer J_DRVL.1
- net 3.0V: no longer I2C.2, I2C_SERVO_DIVER.VDD, RI2CA.1, RI2CL.1
- net ESP_RX_I: now also UART_X.OUTB; no longer UART_X.RXB
- net ESP_TX_O: now also UART_X.OUTA; no longer UART_X.TXB
- net FTDI_RX_I: now also UART_X.INB; no longer UART_X.RXA
- net FTDI_TX_0: now also UART_X.INA; no longer UART_X.TXA
- net GND: no longer D4.VSS, D5.VSS, I2C.1, I2C_SERVO_DIVER.A0, I2C_SERVO_DIVER.A1, I2C_SERVO_DIVER.A2, I2C_SERVO_DIVER.A3, I2C_SERVO_DIVER.A4, I2C_SERVO_DIVER.A5, I2C_SERVO_DIVER.GND, J_EXT_CLK.1
- net N$10: now also BP_P1.1
- net N$11: now also BP_P2.2, BP_P3.1
- net N$12: now also BP_P3.2, WS_OUT.2; no longer D4.DIN
- net N$3: now also BP_P1.2, BP_P2.1
- net VSUPPLY: no longer D4.VDD, D5.VDD
Other:
- moved on the sheet: NM_RX, NM_TX, R_RXH, R_RXL, R_TXH, R_TXL
