File: land-shark-controller/hardware/v2-landshark-handheld-controller.sch (EAGLE design)
At the start: 7 parts

Commit message: Added shark images to BITE and DANCE PARTY. Board file ready for gerberizing.
Parts:
- BITE: value (none) -> BUTTON_PASSIVE_12MM_BITE; device PatternAgents-TouchWidgets:BUTTON_PASSIVE12MM -> PatternAgents-TouchWidgets:BUTTON_PASSIVE_12MM_BITE
- DANCE: value (none) -> BUTTON_PASSIVE_12MM_DANCE; device PatternAgents-TouchWidgets:BUTTON_PASSIVE12MM -> PatternAgents-TouchWidgets:BUTTON_PASSIVE_12MM_DANCE
Changed lines of the file:
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@@
 <part name="BOTTOM" library="PatternAgents-TouchWidgets" deviceset="SLIDER_PASSIVE_1SEG" device=""/>
 <part name="RIGHT" library="PatternAgents-TouchWidgets" deviceset="SLIDER_PASSIVE_1SEG" device=""/>
-<part name="DANCE" library="PatternAgents-TouchWidgets" deviceset="BUTTON_PASSIVE" device="12MM"/>
-<part name="BITE" library="PatternAgents-TouchWidgets" deviceset="BUTTON_PASSIVE" device="12MM"/>
+<part name="DANCE" library="PatternAgents-TouchWidgets" deviceset="BUTTON_PASSIVE_12MM_DANCE" device="" value=""/>
+<part name="BITE" library="PatternAgents-TouchWidgets" deviceset="BUTTON_PASSIVE_12MM_BITE" device="" value=""/>
 </parts>
 <sheets>
@@
 <instance part="BOTTOM" gate="SL1" x="109.22" y="68.58" rot="MR0"/>
 <instance part="RIGHT" gate="SL1" x="109.22" y="53.34" rot="MR0"/>
-<instance part="DANCE" gate="B1" x="157.48" y="81.28" rot="MR0"/>
-<instance part="BITE" gate="B1" x="157.48" y="53.34" rot="MR0"/>
+<instance part="DANCE" gate="G$1" x="157.48" y="81.28" rot="MR0"/>
+<instance part="BITE" gate="G$1" x="157.48" y="53.34" rot="MR0"/>
 </instances>
 <busses>
@@
 <wire x1="129.54" y1="78.74" x2="129.54" y2="53.34" width="0.1524" layer="91"/>
 <wire x1="129.54" y1="53.34" x2="142.24" y2="53.34" width="0.1524" layer="91"/>
-<pinref part="BITE" gate="B1" pin="BUTTON"/>
+<pinref part="BITE" gate="G$1" pin="BUTTON"/>
 </segment>
 </net>
@@
 <wire x1="76.2" y1="63.5" x2="76.2" y2="81.28" width="0.1524" layer="91"/>
 <wire x1="76.2" y1="81.28" x2="142.24" y2="81.28" width="0.1524" layer="91"/>
-<pinref part="DANCE" gate="B1" pin="BUTTON"/>
+<pinref part="DANCE" gate="G$1" pin="BUTTON"/>
 </segment>
 </net>
