File: land-shark-controller/hardware/v3-landshark-handheld-controller.brd (EAGLE design)
At the start: 104 x 50.8 mm, 10 parts

Commit message: Added v3 gerbers, final board. Added 7-pin breakout as per feeeeture creeeeep. Use the gerbers, I took some silk off the top layer.
Parts:
- J1: value (none) -> BREAKOUT; device SparkFun-Connectors:1X06_LOCK_LONGPADS -> SparkFun-Connectors:1X07_LOCK_LONGPADS
- moved J1 12.7 mm to (51.3, 45.1), turned to 180 degrees
Connections:
- new net DIG_IO: J1.5, TEENSY3.6
- net GND: now also J1.6; no longer J1.2
- net SPI_CS: now also J1.4; no longer J1.3
- net SPI_DIN: now also J1.2; no longer J1.5
- net SPI_DOUT: now also J1.3; no longer J1.4
- net SPI_SCK: now also J1.1; no longer J1.6
- net VIN: now also J1.7; no longer J1.1
Routing:
- net DIG_IO: track 0.00 -> 35.2 mm
- net VIN: track 75.1 -> 77.2 mm
Other:
- board text added: "IO"
