File: landshark_bot/base.brd (EAGLE design)
At the start: 64.8 x 57.2 mm, 57 parts

Commit message: Preleminary layout for redoing in shark form factor
Parts:
- added LEFT-DRIVE-SERVO: (no value), tekdemo:MICROSERVO-HORIZONTAL
- added RIGHT-DRIVE-SERVO: RIGHT-DRIVE-SERVO, tekdemo:MICROSERVO-HORIZONTAL-FLIPPED
- added SERVO-BITE, SERVO-LEFTFIN, SERVO-RIGHTFIN, SERVO-TAIL: (no value), tekdemo:MICROSERVER-VERTICAL
- BTN_PROG, BTN_RST: value BUTTONSMD_BUTTON -> BUTTONPJRC; device tekdemo:SMD_BUTTON -> tekdemo:BUTTON-PJRC
- moved LOGO1 62.5 mm to (118.4, 25.7)
- moved X1 5.85 mm to (69.8, 59.4)
- moved BTN_PROG 5.33 mm to (87.4, 66.0)
- moved C_S1 4.93 mm to (67.3, 46.0), turned to 90 degrees
- moved C_S2 2.17 mm to (69.3, 46.0), turned to 90 degrees
- moved BITE 1.78 mm to (66.8, 40.1)
- moved FIN_R 1.78 mm to (66.8, 35.1)
- moved TAIL 1.78 mm to (66.8, 37.6)
- moved C_S3 1.55 mm to (71.6, 46.0), turned to 90 degrees
- moved BP_P1 1.02 mm to (92.7, 47.5), turned to 220 degrees
- moved BP_P2 0.96 mm to (92.8, 39.8), turned to 220 degrees
- moved BP_P3 0.57 mm to (93.0, 32.0), turned to 220 degrees
Connections:
- net BOOTLOADER: now also BTN_PROG.A1, BTN_PROG.A2; no longer BTN_PROG.P$1, BTN_PROG.P$2
- net GND: now also BTN_PROG.B1, BTN_PROG.B2, BTN_RST.B1, BTN_RST.B2; no longer BTN_PROG.P$3, BTN_PROG.P$4, BTN_RST.P$3, BTN_RST.P$4
- net RESET: now also BTN_RST.A1, BTN_RST.A2; no longer BTN_RST.P$1, BTN_RST.P$2
Routing:
- net 3.0V: track 95.6 -> 0.00 mm, vias 6 -> 0
- net VSUPPLY: track 89.0 -> 0.00 mm, vias 15 -> 0
- net GND: track 86.4 -> 0.00 mm, vias 46 -> 0
- net 5V: track 70.8 -> 0.00 mm, vias 13 -> 0
- net 16: track 47.8 -> 0.00 mm, vias 1 -> 0
- net RESET: track 45.8 -> 0.00 mm, vias 2 -> 0
- net 14: track 43.9 -> 0.00 mm, vias 2 -> 0
- net 4: track 41.2 -> 0.00 mm
- net 12: track 40.4 -> 0.00 mm, vias 2 -> 0
- net WAFFLE: track 35.0 -> 0.00 mm
- net 13: track 34.1 -> 0.00 mm, vias 2 -> 0
- net BOOTLOADER: track 31.9 -> 0.00 mm, vias 4 -> 0
- net N$17: track 30.5 -> 0.00 mm, vias 0 -> 3
- net 5: track 29.2 -> 0.00 mm
- net ESP_TX_O: track 25.6 -> 0.00 mm
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- removed copper zone on layer 1, net 5V
- removed copper zone on layer 16, net 5V
- removed copper zone on layer 1, net GND
- removed copper zone on layer 1, net VSUPPLY
- removed copper zone on layer 16, net VSUPPLY
Other:
- board size 64.8 x 57.2 mm -> 250.2 x 108 mm
- board text added: "CENTER"
- board text added: "CUT OUT"
- board text added: "INNER"
- board text added: "LAN'd Shark V3 25-AUG-2015"
- board text added: "OUTSIDE"
- board text removed: "LAN'd Shark V1 Proto 13-JULY-2015"

Commit message: Shark layout partly determined
Parts:
- removed JP1: (no value), SparkFun-Connectors:JST-2-PTH
- removed JP2: (no value), SparkFun-Connectors:1X02_LOCK
- added BAT1: (no value), SparkFun-Electromechanical:BATTERY_18650-HOLDER
- added BAT2: (no value), SparkFun-Electromechanical:BATTERY-AA
- moved R_RST 86.7 mm to (6.10, 50.8), turned to 180 degrees
- moved BTN_RST 84.6 mm to (6.10, 48.0), flipped to the bottom
- moved X1 80.0 mm to (11.2, 5.08), turned to 180 degrees
- moved R_BOOT 76.6 mm to (14.2, 50.8), turned to 180 degrees
- moved BTN_PROG 75.3 mm to (14.2, 48.0), flipped to the bottom
- moved LEFT-DRIVE-SERVO 67.3 mm to (23.4, 30.5)
- moved SERVO-TAIL 66.6 mm to (66.0, 17.8), turned to 0 degrees
- moved SERVO-BITE 66.3 mm to (-17.0, 17.8), turned to 0 degrees
- moved SERVO-LEFTFIN 61.0 mm to (32.8, 11.4)
- moved SERVO-RIGHTFIN 61.0 mm to (32.8, 24.1)
- moved RIGHT-DRIVE-SERVO 54.6 mm to (0.51, 17.8)
- moved R_LCHRG 53.6 mm to (91.2, 20.6)
- moved R_LDONE 53.6 mm to (91.2, 23.1)
- moved R_LED 53.6 mm to (91.2, 28.2)
- moved R_LPWR 53.6 mm to (91.2, 25.7)
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Connections:
- net GND: now also BAT1.GND@1, BAT2.GND@1; no longer JP1.2, JP2.2
- net VBAT: now also BAT1.PWR@1, BAT2.PWR@1; no longer JP1.1, JP2.1
Routing:
- net N$30: track 12.8 -> 0.00 mm, vias 2 -> 0
- net N$29: track 9.69 -> 0.00 mm, vias 2 -> 0
- net N$28: track 6.60 -> 0.00 mm, vias 2 -> 0
Other:
- board size 250.2 x 108 mm -> 479.6 x 158.1 mm
