File: landshark_bot/base.sch (EAGLE design)
At the start: 57 parts

Commit message: Preleminary layout for redoing in shark form factor
Parts:
- BTN_PROG, BTN_RST: value BUTTONSMD_BUTTON -> BUTTONPJRC; device tekdemo:BUTTONSMD_BUTTON -> tekdemo:BUTTONPJRC
Changed lines of the file:
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@@
 <layer number="19" name="Unrouted" color="6" fill="1" visible="no" active="no"/>
 <layer number="20" name="Dimension" color="15" fill="1" visible="no" active="no"/>
-<layer number="21" name="tPlace" color="7" fill="1" visible="no" active="no"/>
-<layer number="22" name="bPlace" color="7" fill="1" visible="no" active="no"/>
+<layer number="21" name="tPlace" color="16" fill="1" visible="no" active="no"/>
+<layer number="22" name="bPlace" color="14" fill="1" visible="no" active="no"/>
 <layer number="23" name="tOrigins" color="15" fill="1" visible="no" active="no"/>
 <layer number="24" name="bOrigins" color="15" fill="1" visible="no" active="no"/>
@@
 <layer number="49" name="Reference" color="7" fill="1" visible="no" active="no"/>
 <layer number="50" name="dxf" color="7" fill="1" visible="no" active="no"/>
-<layer number="51" name="tDocu" color="7" fill="1" visible="no" active="no"/>
+<layer number="51" name="tDocu" color="6" fill="1" visible="no" active="no"/>
 <layer number="52" name="bDocu" color="7" fill="1" visible="no" active="no"/>
 <layer number="53" name="tGND_GNDA" color="7" fill="9" visible="no" active="no"/>
@@
 <part name="X1" library="adafruit" deviceset="ESP-12" device=""/>
 <part name="UART_X" library="tekdemo" deviceset="UART_SWITCHER" device="0603"/>
-<part name="BTN_RST" library="tekdemo" deviceset="BUTTON" device="SMD_BUTTON"/>
-<part name="BTN_PROG" library="tekdemo" deviceset="BUTTON" device="SMD_BUTTON"/>
+<part name="BTN_RST" library="tekdemo" deviceset="BUTTON" device="PJRC" value="BUTTONPJRC"/>
+<part name="BTN_PROG" library="tekdemo" deviceset="BUTTON" device="PJRC" value="BUTTONPJRC"/>
 <part name="DRV_L" library="SparkFun-Connectors" deviceset="M03" device="LOCK"/>
 <part name="DRV_R" library="SparkFun-Connectors" deviceset="M03" device="LOCK"/>

Commit message: Shark layout partly determined
Parts:
- removed JP1: (no value), SparkFun-Connectors:M02JST-PTH-2
- removed JP2: (no value), SparkFun-Connectors:M02LOCK
- added BAT1: (no value), SparkFun-Electromechanical:BATTERY18650
- added BAT2: (no value), SparkFun-Electromechanical:BATTERYAA
Connections:
- net GND: now also BAT1.-, BAT2.-; no longer JP1.2, JP2.2
- net VBAT: now also BAT1.+, BAT2.+; no longer JP1.1, JP2.1
Changed lines of the file:
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@@
 <part name="C_BLKY" library="tekdemo" deviceset="CAP" device="UNIVERSAL" value="0.1uF"/>
 <part name="R_BLNK" library="tekdemo" deviceset="RESISTOR" device="UNIVERSAL" value="50"/>
-<part name="JP1" library="SparkFun-Connectors" deviceset="M02" device="JST-PTH-2"/>
-<part name="JP2" library="SparkFun-Connectors" deviceset="M02" device="LOCK"/>
 <part name="BP_P1" library="SparkFun-Passives" deviceset="JUMPER-PAD-2-NO" device="YES_SILK" value=""/>
 <part name="BP_P2" library="SparkFun-Passives" deviceset="JUMPER-PAD-2-NO" device="YES_SILK" value=""/>
 <part name="BP_P3" library="SparkFun-Passives" deviceset="JUMPER-PAD-2-NO" device="YES_SILK" value=""/>
+<part name="BAT1" library="SparkFun-Electromechanical" deviceset="BATTERY" device="18650"/>
+<part name="BAT2" library="SparkFun-Electromechanical" deviceset="BATTERY" device="AA"/>
 </parts>
 <sheets>
@@
 <instance part="C_BLKY" gate="G$1" x="182.88" y="33.02" rot="MR180"/>
 <instance part="R_BLNK" gate="G$1" x="205.74" y="40.64"/>
-<instance part="JP1" gate="G$1" x="43.18" y="-38.1" rot="R180"/>
-<instance part="JP2" gate="G$1" x="55.88" y="-38.1" rot="R180"/>
 <instance part="BP_P1" gate="G$1" x="220.98" y="35.56"/>
 <instance part="BP_P2" gate="G$1" x="248.92" y="35.56"/>
 <instance part="BP_P3" gate="G$1" x="274.32" y="35.56"/>
+<instance part="BAT1" gate="G$1" x="25.4" y="-40.64" rot="R270"/>
+<instance part="BAT2" gate="G$1" x="20.32" y="-40.64" rot="R270"/>
 </instances>
 <busses>
@@
 </segment>
 <segment>
-<wire x1="10.16" y1="-43.18" x2="15.24" y2="-43.18" width="0.2032" layer="91"/>
-<label x="15.24" y="-43.18" size="1.778" layer="95" xref="yes"/>
+<wire x1="10.16" y1="-43.18" x2="10.16" y2="-45.72" width="0.2032" layer="91"/>
+<wire x1="10.16" y1="-45.72" x2="20.32" y2="-45.72" width="0.2032" layer="91"/>
+<label x="25.4" y="-45.72" size="1.778" layer="95" xref="yes"/>
 <pinref part="C_BAT" gate="G$1" pin="2"/>
-<pinref part="JP1" gate="G$1" pin="2"/>
-<wire x1="15.24" y1="-43.18" x2="17.78" y2="-40.64" width="0.2032" layer="91"/>
-<wire x1="17.78" y1="-40.64" x2="35.56" y2="-40.64" width="0.2032" layer="91"/>
-<pinref part="JP2" gate="G$1" pin="2"/>
-<wire x1="35.56" y1="-40.64" x2="48.26" y2="-40.64" width="0.2032" layer="91"/>
+<pinref part="BAT1" gate="G$1" pin="-"/>
+<pinref part="BAT2" gate="G$1" pin="-"/>
+<wire x1="20.32" y1="-45.72" x2="25.4" y2="-45.72" width="0.2032" layer="91"/>
+<junction x="20.32" y="-45.72"/>
 </segment>
 </net>
@@
 <wire x1="-10.16" y1="-38.1" x2="-10.16" y2="-35.56" width="0.2032" layer="91"/>
 <wire x1="-10.16" y1="-35.56" x2="10.16" y2="-35.56" width="0.2032" layer="91"/>
-<label x="15.24" y="-35.56" size="1.778" layer="95" xref="yes"/>
+<label x="25.4" y="-35.56" size="1.778" layer="95" xref="yes"/>
 <pinref part="C_BAT" gate="G$1" pin="1"/>
-<wire x1="10.16" y1="-35.56" x2="15.24" y2="-35.56" width="0.2032" layer="91"/>
 <junction x="10.16" y="-35.56"/>
 <junction x="-10.16" y="-35.56"/>
 <junction x="-10.16" y="-33.02"/>
 <junction x="-10.16" y="-38.1"/>
-<pinref part="JP1" gate="G$1" pin="1"/>
-<wire x1="15.24" y1="-35.56" x2="17.78" y2="-38.1" width="0.2032" layer="91"/>
-<wire x1="17.78" y1="-38.1" x2="35.56" y2="-38.1" width="0.2032" layer="91"/>
-<pinref part="JP2" gate="G$1" pin="1"/>
-<wire x1="35.56" y1="-38.1" x2="48.26" y2="-38.1" width="0.2032" layer="91"/>
-</segment>
-</net>
+<wire x1="10.16" y1="-35.56" x2="20.32" y2="-35.56" width="0.2032" layer="91"/>
+<pinref part="BAT1" gate="G$1" pin="+"/>
+<pinref part="BAT2" gate="G$1" pin="+"/>
+<wire x1="20.32" y1="-35.56" x2="25.4" y2="-35.56" width="0.2032" layer="91"/>
+<junction x="20.32" y="-35.56"/>
+</segment>
+</net>
