File: landshark_bot/chassis.brd (EAGLE design)
At the start: 242.4 x 158.1 mm, 20 parts

Commit message: Updated routing and shuffled things a bit, tail
Parts:
- removed LEFT-DRIVE-SERVO: (no value), tekdemo:MICROSERVO-HORIZONTAL
- removed RIGHT-DRIVE-SERVO: RIGHT-DRIVE-SERVO, tekdemo:MICROSERVO-HORIZONTAL-FLIPPED
- added SERVO-LEFT-DRIVE: RIGHT-DRIVE-SERVO, tekdemo:MICROSERVO-HORIZONTAL-FLIPPED
- added SERVO-RIGHT-DRIVE: (no value), tekdemo:MICROSERVO-HORIZONTAL
- moved SERVO-LEFTFIN 38.2 mm to (85.1, 9.14), turned to 0 degrees
- moved SERVO-TAIL 38.2 mm to (113.8, 34.3), turned to 270 degrees
- moved BP_P4 2.34 mm to (29.2, 37.1)
- moved D4 2.34 mm to (29.2, 37.1)
- moved BP_P2 1.63 mm to (29.2, 8.89)
- moved D2 1.63 mm to (29.2, 8.89)
- moved SERVO-BITE 1.27 mm to (47.0, 11.4)
Routing:
- net GND: track 28.9 -> 13.9 mm, vias 7 -> 19
- net VSUPPLY: track 208.3 -> 215.2 mm
- net N$4: track 59.2 -> 64.8 mm
- net N$3: track 61.1 -> 65.5 mm
- net N$12: track 37.6 -> 35.4 mm
- net N$11: track 35.1 -> 33.4 mm
Other:
- board size 242.4 x 158.1 mm -> 160.5 x 43.9 mm
- board text added: "LAN'd Shark Chassis V1 01-Sep-2015"
- board text removed: "LAN'd Shark V3 25-AUG-2015"
