File: landshark_bot/brains.brd (EAGLE design)
At the start: 479.6 x 158.1 mm, 63 parts

Commit message: Finished rerouting the brain board!
Parts:
- removed BAT1: (no value), SparkFun-Electromechanical:BATTERY_18650-HOLDER
- removed BP_P1, BP_P2, BP_P3, JP_LS_BP_RX, J_LS_BP_TX: (no value), SparkFun-Passives:PAD-JUMPER-2-NO_YES_SILK
- removed C_BLKY: 0.1uF, tekdemo:0402-0603-0805-UNIVERSAL
- removed D1, D2, D3: (no value), tekdemo:WS2812B
- removed LEFT-DRIVE-SERVO: (no value), tekdemo:MICROSERVO-HORIZONTAL
- removed NM_RX, NM_TX: MOSFET-NCHANNELSMD, tekdemo:SOT23-3
- removed RIGHT-DRIVE-SERVO: RIGHT-DRIVE-SERVO, tekdemo:MICROSERVO-HORIZONTAL-FLIPPED
- removed R_BLNK: 50, tekdemo:0402-0603-0805-UNIVERSAL
- removed R_RXH, R_RXL, R_TXH, R_TXL: (no value), tekdemo:0402-0603-0805-UNIVERSAL
- removed SERVO-BITE, SERVO-LEFTFIN, SERVO-RIGHTFIN, SERVO-TAIL: (no value), tekdemo:MICROSERVER-VERTICAL
- C_S1: device tekdemo:0402-0603-0805-UNIVERSAL -> tekdemo:1210
- moved BAT2 192.4 mm to (25.4, 26.7), flipped to the bottom, turned to 270 degrees
- moved LOGO1 87.6 mm to (36.1, 39.6), flipped to the bottom
- moved C_S3 76.4 mm to (53.1, 15.0), turned to 0 degrees
- moved C_S2 73.6 mm to (53.1, 16.8), turned to 0 degrees
- moved C_BAT 73.5 mm to (25.4, 13.0), turned to 0 degrees
- moved R_PD1 72.1 mm to (24.1, 17.5), turned to 180 degrees
- moved C_5V 72.0 mm to (29.7, 9.91), turned to 270 degrees
- moved C_S1 70.5 mm to (53.1, 19.1), turned to 180 degrees
- moved R_PD2 70.2 mm to (24.1, 19.8), turned to 180 degrees
- moved IC_LIPO 67.8 mm to (30.0, 16.0), turned to 180 degrees
- moved C_SUP 66.0 mm to (32.5, 9.91)
- moved R_LED 58.8 mm to (35.3, 9.91), turned to 270 degrees
- moved FTDI 56.5 mm to (16.8, 24.6)
- moved R_PD3 56.2 mm to (36.1, 22.9), turned to 0 degrees
- moved R_LPWR 56.0 mm to (36.1, 16.0), turned to 180 degrees
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Connections:
- removed net FTDI_RX_I_HV: FTDI.3, JP_LS_BP_RX.1, NM_RX.3, R_RXH.-
- removed net FTDI_TX_0_HV: FTDI.2, J_LS_BP_TX.1, NM_TX.3, R_TXH.-
- removed net N$11: BP_P2.2, BP_P3.1, D2.2, D3.4
- removed net N$12: BP_P3.2, D3.2, WS_OUT.2
- removed net N$21: IC_LIPO.6, R_LDONE.-
- new net CHARGE_DONE: IC_LIPO.6, R_LDONE.-, X1.2
- net 3.0V: now also R_BOOT.+, R_RST.+; no longer C_ESP1.-, C_ESP2.-, R_BOOT.-, R_RST.-, R_RXL.+, R_TXL.+
- net 5V: no longer LED_CHRG.+, LED_DONE.+, LED_PWR.+, NM_RX.1, NM_TX.1, R_RXH.+, R_TXH.+
- net BLINKY: now also WS_OUT.2; no longer R_BLNK.+
- net BOOTLOADER: now also R_BOOT.-; no longer R_BOOT.+
- net FTDI_RX_I: now also FTDI.3; no longer JP_LS_BP_RX.2, NM_RX.2, R_RXL.-
- net FTDI_TX_0: now also FTDI.2; no longer J_LS_BP_TX.2, NM_TX.2, R_TXL.-
- net GND: now also C_BAT.-, C_S1.1, C_SUP.-; no longer BAT1.GND@1, C_BAT.+, C_BLKY.-, C_ESP1.+, C_ESP2.+, C_S1.-, C_SUP.+, D1.3, D2.3, D3.3
- net N$10: now also C_ESP1.+, C_ESP2.+; no longer BP_P1.1, D1.4, R_BLNK.-
- net N$3: now also C_ESP1.-, C_ESP2.-; no longer BP_P1.2, BP_P2.1, D1.2, D2.4
- net RESET: now also R_RST.-; no longer R_RST.+
- net VBAT: now also C_BAT.+; no longer BAT1.PWR@1, C_BAT.-
- net VSUPPLY: now also C_S1.2, C_SUP.+, LED_CHRG.+, LED_DONE.+, LED_PWR.+; no longer C_BLKY.+, C_S1.+, C_SUP.-, D1.1, D2.1, D3.1
Routing:
- net VSUPPLY: track 0.00 -> 56.2 mm, vias 0 -> 1
- net BLINKY: track 0.00 -> 50.8 mm
- net GND: track 0.00 -> 49.0 mm, vias 0 -> 24
- net BOOTLOADER: track 0.00 -> 47.6 mm
- net 3.0V: track 0.00 -> 44.4 mm, vias 0 -> 3
- net FTDI_RX_I: track 0.00 -> 29.0 mm, vias 0 -> 1
- net FTDI_TX_0: track 0.00 -> 22.3 mm, vias 0 -> 1
- net 4: track 0.00 -> 19.6 mm
- net 5V: track 0.00 -> 17.0 mm, vias 0 -> 3
- net 5: track 0.00 -> 16.7 mm
- net 16: track 0.00 -> 16.0 mm
- net RESET: track 0.00 -> 15.9 mm
- net VBAT: track 0.00 -> 15.0 mm, vias 0 -> 5
- net CHARGE_DONE: track 0.00 -> 14.5 mm, vias 0 -> 2
- net 14: track 0.00 -> 14.1 mm
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- added copper zone on layer 1, net 5V
- added copper zone on layer 1, net GND
- added copper zone on layer 1, net VBAT
- added copper zone on layer 16, net VBAT
- added copper zone on layer 1, net VSUPPLY
- removed copper zone on layer 1, net N$15
Other:
- board size 479.6 x 158.1 mm -> 479.6 x 167.1 mm
- board text added: "5V"
- board text added: "BITE TAIL R FIN L FIN R DRV L DRV"
- board text added: "LAN'd Shark Brains V3 1-SEP-2015"
- board text removed: "CENTER"
- board text removed: "CUT OUT"
- board text removed: "INNER"
- board text removed: "LAN'd Shark V3 25-AUG-2015"
- board text removed: "OUTSIDE"

Commit message: As ordered for Maker Faire
Parts:
- moved C_ESP1 14.7 mm to (47.8, 50.3)
- moved C_ESP2 14.7 mm to (47.8, 52.6)
Other:
- board size 479.6 x 167.1 mm -> 235.1 x 167.1 mm
- board text added: "ONLY HERE TO CONFUSE KELLY -->"
- board text added: "SHARK BRAINS!"
