File: landshark_bot/brains.sch (EAGLE design)
At the start: 57 parts

Commit message: Finished rerouting the brain board!
Parts:
- removed BAT1: (no value), SparkFun-Electromechanical:BATTERY18650
- removed BP_P1, BP_P2, BP_P3, JP_LS_BP_RX, J_LS_BP_TX: JUMPER-PAD-2-NOYES_SILK, SparkFun-Passives:JUMPER-PAD-2-NOYES_SILK
- removed C_BLKY: 0.1uF, tekdemo:CAPUNIVERSAL
- removed D1, D2, D3: (no value), tekdemo:WS2812B
- removed NM_RX, NM_TX: MOSFET-NCHANNELSMD, tekdemo:MOSFET-NCHANNELSMD
- removed R_BLNK: 50, tekdemo:RESISTORUNIVERSAL
- removed R_RXH, R_RXL, R_TXH, R_TXL: (no value), tekdemo:RESISTORUNIVERSAL
- C_S1: device tekdemo:CAPUNIVERSAL -> tekdemo:CAP1210
Connections:
- removed net FTDI_RX_I_HV: FTDI.3, JP_LS_BP_RX.1, NM_RX.D, R_RXH.2
- removed net FTDI_TX_0_HV: FTDI.2, J_LS_BP_TX.1, NM_TX.D, R_TXH.2
- removed net N$11: BP_P2.2, BP_P3.1, D2.DOUT, D3.DIN
- removed net N$12: BP_P3.2, D3.DOUT, WS_OUT.2
- removed net N$21: IC_LIPO./PG, R_LDONE.2
- new net CHARGE_DONE: IC_LIPO./PG, R_LDONE.2, X1.ADC
- net 3.0V: now also R_BOOT.1, R_RST.1; no longer C_ESP1.1, C_ESP2.1, R_BOOT.2, R_RST.2, R_RXL.1, R_TXL.1
- net 5V: no longer LED_CHRG.A, LED_DONE.A, LED_PWR.A, NM_RX.G, NM_TX.G, R_RXH.1, R_TXH.1
- net BLINKY: now also WS_OUT.2; no longer R_BLNK.1
- net BOOTLOADER: now also R_BOOT.2; no longer R_BOOT.1
- net FTDI_RX_I: now also FTDI.3; no longer JP_LS_BP_RX.2, NM_RX.S, R_RXL.2
- net FTDI_TX_0: now also FTDI.2; no longer J_LS_BP_TX.2, NM_TX.S, R_TXL.2
- net GND: now also C_BAT.1, C_SUP.1; no longer BAT1.-, C_BAT.2, C_BLKY.1, C_ESP1.2, C_ESP2.2, C_SUP.2, D1.VSS, D2.VSS, D3.VSS
- net N$10: now also C_ESP1.2, C_ESP2.2; no longer BP_P1.1, D1.DIN, R_BLNK.2
- net N$3: now also C_ESP1.1, C_ESP2.1; no longer BP_P1.2, BP_P2.1, D1.DOUT, D2.DIN
- net RESET: now also R_RST.2; no longer R_RST.1
- net VBAT: now also C_BAT.2; no longer BAT1.+, C_BAT.1
- net VSUPPLY: now also C_SUP.2, LED_CHRG.A, LED_DONE.A, LED_PWR.A; no longer C_BLKY.2, C_SUP.1, D1.VDD, D2.VDD, D3.VDD
Other:
- note added: "BYPASS CAPS LEFT OUT DUE TO ESP HAVING DEDICATED REGULAR, CONVENIENTLY PLACED NEAR THE VCC PIN"
- note added: "located on chassis"
- note removed: "LEVEL SHIFTING BYPASS JUMPERS"
- note removed: "OPTIMAL: add auto-reset when DTR goes down Similar to arduino. Verify via forum somewhere."
- note removed: "TECHNICALLY ONLY ONE LEVEL SHIFTER IS NEEDED"
- note removed: "VERIFY LEVEL SHIFTER RESISTOR VALUES"
- moved on the sheet: C_5V, C_BAT, C_SUP, LED_DONE, LED_PWR, R_BOOT, R_LDONE, R_LPWR, R_RST

Commit message: As ordered for Maker Faire
Other:
- note added: "BYPASS CAPS LEFT OUT DUE TO ESP HAVING DEDICATED REGULATOR, CONVENIENTLY PLACED NEAR THE VCC PIN"
- note removed: "BYPASS CAPS LEFT OUT DUE TO ESP HAVING DEDICATED REGULAR, CONVENIENTLY PLACED NEAR THE VCC PIN"
- moved on the sheet: WS_OUT
Changed lines of the file:
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@@
 <text x="129.54" y="-12.7" size="1.778" layer="94">SERVOS AND MOTION</text>
 <wire x1="170.18" y1="60.96" x2="170.18" y2="-5.08" width="0.2032" layer="94"/>
-<wire x1="170.18" y1="-5.08" x2="360.68" y2="-5.08" width="0.2032" layer="94"/>
-<wire x1="360.68" y1="-5.08" x2="360.68" y2="60.96" width="0.2032" layer="94"/>
-<wire x1="360.68" y1="60.96" x2="170.18" y2="60.96" width="0.2032" layer="94"/>
+<wire x1="170.18" y1="-5.08" x2="248.92" y2="-5.08" width="0.2032" layer="94"/>
+<wire x1="248.92" y1="-5.08" x2="248.92" y2="60.96" width="0.2032" layer="94"/>
+<wire x1="248.92" y1="60.96" x2="170.18" y2="60.96" width="0.2032" layer="94"/>
 <text x="203.2" y="60.96" size="1.778" layer="94">BLINKELNIGHTS</text>
 <text x="-71.12" y="0" size="1.778" layer="91">OPTIMAL:
@@
 IN BOOTLOADER
 SECTION</text>
-<text x="198.12" y="43.18" size="1.778" layer="91">located on chassis</text>
-<text x="116.84" y="68.58" size="1.778" layer="91">BYPASS CAPS LEFT OUT DUE TO ESP HAVING DEDICATED REGULAR,
+<text x="200.66" y="58.42" size="1.778" layer="91">located on chassis</text>
+<text x="116.84" y="68.58" size="1.778" layer="91">BYPASS CAPS LEFT OUT DUE TO ESP HAVING DEDICATED REGULATOR,
  CONVENIENTLY PLACED NEAR THE VCC PIN</text>
 </plain>
@@
 <instance part="BITE" gate="G$1" x="342.9" y="-27.94"/>
 <instance part="VREG_3V" gate="G$1" x="33.02" y="-83.82"/>
-<instance part="WS_OUT" gate="G$1" x="350.52" y="33.02" rot="R180"/>
+<instance part="WS_OUT" gate="G$1" x="238.76" y="33.02" rot="R180"/>
 <instance part="LED" gate="G$1" x="10.16" y="-76.2"/>
 <instance part="R_LED" gate="G$1" x="10.16" y="-88.9" rot="R270"/>
@@
 </segment>
 <segment>
-<label x="180.34" y="25.4" size="1.778" layer="95" rot="R180" xref="yes"/>
-<wire x1="180.34" y1="25.4" x2="342.9" y2="25.4" width="0.2032" layer="91"/>
+<label x="187.96" y="27.94" size="1.778" layer="95" rot="R180" xref="yes"/>
+<wire x1="187.96" y1="27.94" x2="231.14" y2="27.94" width="0.2032" layer="91"/>
 <pinref part="WS_OUT" gate="G$1" pin="3"/>
-<wire x1="342.9" y1="30.48" x2="342.9" y2="25.4" width="0.2032" layer="91"/>
+<wire x1="231.14" y1="30.48" x2="231.14" y2="27.94" width="0.2032" layer="91"/>
 </segment>
 <segment>
@@
 <net name="BLINKY" class="0">
 <segment>
-<wire x1="200.66" y1="40.64" x2="195.58" y2="40.64" width="0.2032" layer="91"/>
-<label x="195.58" y="40.64" size="1.778" layer="95" rot="R180" xref="yes"/>
+<label x="187.96" y="33.02" size="1.778" layer="95" rot="R180" xref="yes"/>
 <pinref part="WS_OUT" gate="G$1" pin="2"/>
-<wire x1="342.9" y1="33.02" x2="200.66" y2="33.02" width="0.2032" layer="91"/>
-<wire x1="200.66" y1="33.02" x2="200.66" y2="40.64" width="0.2032" layer="91"/>
+<wire x1="231.14" y1="33.02" x2="187.96" y2="33.02" width="0.2032" layer="91"/>
 </segment>
 <segment>
@@
 </segment>
 <segment>
-<wire x1="180.34" y1="50.8" x2="342.9" y2="50.8" width="0.2032" layer="91"/>
-<label x="180.34" y="50.8" size="1.778" layer="95" rot="R180" xref="yes"/>
+<wire x1="187.96" y1="38.1" x2="231.14" y2="38.1" width="0.2032" layer="91"/>
+<label x="187.96" y="38.1" size="1.778" layer="95" rot="R180" xref="yes"/>
 <pinref part="WS_OUT" gate="G$1" pin="1"/>
-<wire x1="342.9" y1="35.56" x2="342.9" y2="50.8" width="0.2032" layer="91"/>
-</segment>
-<segment>
+<wire x1="231.14" y1="35.56" x2="231.14" y2="38.1" width="0.2032" layer="91"/>
+</segment>
+<segment>
