File: landshark_bot/fins.brd (EAGLE design)
At the start: 163.3 x 53.6 mm, 6 parts

Commit message: As ordered for Maker Faire
Routing:
- net BITET: track 0.00 -> 1.48 mm
- added copper zone on layer 1, net BITET
Other:
- board size 163.3 x 53.6 mm -> 147.3 x 56.4 mm
- board text removed: "LAN'd Shark Chassis V1 01-Sep-2015"
